Commit message: Update robot and rope assets

File: assets/single_system/arm/AR5V2_L/AR5V2_L.urdf (robot description, URDF)
Before this commit: robot AR5V2_L_arm, 10 links, 9 joints
Joints:
- joint AR5V2_L_arm_joint_6: limit lower=-0.9599 upper=0.9599 effort=19 velocity=4.1887902047863905 -> lower=-1.2 upper=1.2 effort=19 velocity=4.1887902047863905
- joint AR5V2_L_arm_joint_7: limit lower=-0.9599 upper=0.9599 effort=19 velocity=4.1887902047863905 -> lower=-1.2 upper=1.2 effort=19 velocity=4.1887902047863905

File: assets/single_system/arm/AR5V2_R/AR5V2_R.urdf (robot description, URDF)
Before this commit: robot AR5V2_R_arm, 10 links, 9 joints
Joints:
- joint AR5V2_R_arm_joint_6: limit lower=-0.9599 upper=0.9599 effort=19 velocity=4.1887902047863905 -> lower=-1.2 upper=1.2 effort=19 velocity=4.1887902047863905
- joint AR5V2_R_arm_joint_7: limit lower=-0.9599 upper=0.9599 effort=19 velocity=4.1887902047863905 -> lower=-1.2 upper=1.2 effort=19 velocity=4.1887902047863905
