Commit message: feat: 完善物体 usd 生成模块, 支持动态/静态物体的生成 (#18)
closes LinkerOS/scene-replay-sim-Isaac#16

Reviewed-on: https://gitea.linkerhub.work/LinkerOS/scene-replay-sim-Isaac/pulls/18
Co-authored-by: songpengyang <1559265150@qq.com>
Co-committed-by: songpengyang <1559265150@qq.com>

File: assets/rigid_env_objects/workstationV1_armbase/workstationV1_armbase.urdf (robot description, URDF)
Before this commit: robot workstationV1_tablebase_frame, 1 links, 0 joints
Links:
- removed link workstationV1_tablebase_frame
- added link workstationV1_armbase_frame, mass 100.0; collision box size=0.06 0.12 1.1; collision box size=0.625 1.25 0.77

File: assets/rigid_env_objects/workstationV1_tablebase/workstationV1_tablebase.urdf (robot description, URDF)
Before this commit: robot workstationV1_armbase_frame, 1 links, 0 joints
Links:
- removed link workstationV1_armbase_frame
- added link workstationV1_tablebase_frame, mass 100.0; collision box size=0.06 0.12 1.1; collision box size=0.625 1.25 0.77
